Commit message: updated transforms of sensors in urdf files

File: segway_robot/defs/base.urdf (robot description, URDF)
Before this commit: robot base, 13 links, 12 joints
Joints:
- joint R283_hokuyo_laser1_joint: origin xyz=-0.162 -0.062 0 rpy=0 0 0 -> xyz=-0.162 -0.062 0 rpy=0 0 -0.1848
- joint R313_hokuyo_laser2_joint: origin xyz=-0.162 0.283 0 rpy=3.14159 0 0 -> xyz=-0.162 0.283 0 rpy=1.57 -0.05 0
- joint base_footprint_joint: origin xyz=0 0 0.55 rpy=1.57 0 3.14 -> xyz=0 0 0.55 rpy=1.57 0 3.14159

File: segway_robot/defs/sensors.urdf (robot description, URDF)
Before this commit: robot hand, 2 links, 2 joints
Joints:
- joint tilt_laser_joint: origin xyz=-0.056 0.020 0 rpy=-1.57 0 3.14 -> xyz=-0.056 -0.020 0 rpy=-1.57 0 3.14
