Commit message: fixes to segbot xacro

File: segway_robot/gazebo/gazebo.urdf.xacro (robot description, xacro)
@@ -1,18 +1,4 @@
-<xml version="1.0"?>
+<?xml version="1.0"?>
 <robot xmlns:xacro="http://ros.org/wiki/xacro">
-    <!-- From old Gazebo configuration
-    <material name="Blue">
-        <color rgba="0.0 0.0 0.8 1.0"/>
-    </material>
-    <material name="Green">
-        <color rgba="0.0 0.8 0.0 1.0"/>
-    </material>
-    <material name="Red">
-        <color rgba="0.8 0.0 0.0 1.0"/>
-    </material>
-    <material name="White">
-        <color rgba="0.0 0.0 0.0 1.0"/>
-    </material>
-    -->
     <gazebo>
         <static>false</static>

File: segway_robot/urdf/base.gazebo.xacro (robot description, xacro)
@@ -52,5 +52,5 @@
                 <robotBaseFrame>base_footprint</robotBaseFrame>
             </plugin>
-            <plugin name="p3d_base_controller" plugin="libgazebo_ros_p3d.so">
+            <plugin name="p3d_base_controller" filename="libgazebo_ros_p3d.so">
                 <alwaysOn>true</alwaysOn>
                 <robotNamespace></robotNamespace>

File: segway_robot/urdf/base.transmission.xacro (robot description, xacro)
@@ -7,9 +7,9 @@
                 <hardwareInterface>EffortJointInterface</hardwareInterface>
             </joint>
+            <actuator name="segway_left_wheel_motor">
+                <hardwareInterface>EffortJointInterface</hardwareInterface>
+                <mechanicalReduction>1.0</mechanicalReduction>
+            </actuator>
         </transmission>
-        <actuator name="segway_left_wheel_motor">
-            <hardwareInterface>EffortJointInterface</hardwareInterface>
-            <mechanicalReduction>1.0</mechanicalReduction>
-        </actuator>
         <transmission name="segway_right_wheel_trans">
             <type>transmission_interface/SimpleTransmission</type>
@@ -17,9 +17,9 @@
                 <hardwareInterface>EffortJointInterface</hardwareInterface>
             </joint>
+            <actuator name="segway_right_wheel_motor">
+                <hardwareInterface>EffortJointInterface</hardwareInterface>
+                <mechanicalReduction>1.0</mechanicalReduction>
+            </actuator>
         </transmission>
-        <actuator name="segway_right_wheel_motor">
-            <hardwareInterface>EffortJointInterface</hardwareInterface>
-            <mechanicalReduction>1.0</mechanicalReduction>
-        </actuator>
         <transmission name="segway_trailer_wheel_caster_trans">
             <type>transmission_interface/SimpleTransmission</type>
@@ -27,9 +27,9 @@
                 <hardwareInterface>EffortJointInterface</hardwareInterface>
             </joint>
+            <actuator name="segway_trailer_wheel_caster_motor">
+                <hardwareInterface>EffortJointInterface</hardwareInterface>
+                <mechanicalReduction>1.0</mechanicalReduction>
+            </actuator>
         </transmission>
-        <actuator name="segway_trailer_wheel_caster_motor">
-            <hardwareInterface>EffortJointInterface</hardwareInterface>
-            <mechanicalReduction>1.0</mechanicalReduction>
-        </actuator>
         <transmission name="segway_trailer_wheel_trans">
             <type>transmission_interface/SimpleTransmission</type>
@@ -37,9 +37,9 @@
                 <hardwareInterface>EffortJointInterface</hardwareInterface>
             </joint>
+            <actuator name="segway_trailer_wheel_motor">
+                <hardwareInterface>EffortJointInterface</hardwareInterface>
+                <mechanicalReduction>1.0</mechanicalReduction>
+            </actuator>
         </transmission>
-        <actuator name="segway_trailer_wheel_motor">
-            <hardwareInterface>EffortJointInterface</hardwareInterface>
-            <mechanicalReduction>1.0</mechanicalReduction>
-        </actuator>
         <transmission name="R283_hokuyo_laser1_trans">
             <type>transmission_interface/SimpleTransmission</type>
@@ -47,9 +47,9 @@
                 <hardwareInterface>EffortJointInterface</hardwareInterface>
             </joint>
+            <actuator name="R283_hokuyo_laser1_motor">
+                <hardwareInterface>EffortJointInterface</hardwareInterface>
+                <mechanicalReduction>1.0</mechanicalReduction>
+            </actuator>
         </transmission>
-        <actuator name="R283_hokuyo_laser1_motor">
-            <hardwareInterface>EffortJointInterface</hardwareInterface>
-            <mechanicalReduction>1.0</mechanicalReduction>
-        </actuator>
         <transmission name="R313_hokuyo_laser2_trans">
             <type>transmission_interface/SimpleTransmission</type>
@@ -57,9 +57,9 @@
                 <hardwareInterface>EffortJointInterface</hardwareInterface>
             </joint>
+            <actuator name="R313_hokuyo_laser2_motor">
+                <hardwareInterface>EffortJointInterface</hardwareInterface>
+                <mechanicalReduction>1.0</mechanicalReduction>
+            </actuator>
         </transmission>
-        <actuator name="R313_hokuyo_laser2_motor">
-            <hardwareInterface>EffortJointInterface</hardwareInterface>
-            <mechanicalReduction>1.0</mechanicalReduction>
-        </actuator>
     </xacro:macro>
 </robot>

File: segway_robot/urdf/base.urdf.xacro (robot description, xacro)
@@ -5,8 +5,8 @@
     <xacro:macro name="base" params="name">
         <!-- JOINT LIMIT VALUES FOR EFFORT AND VELOCITY NEED TO BE ADDED FOR
-        <!-- REVOLUTE AND CONTINUOUS JOINTS -->
+        REVOLUTE AND CONTINUOUS JOINTS
+        -->
         <!-- base_footprint is a fictitious link(frame) that is on the ground
-        <!-- right below base_link origin, navigation stack depends on this
-        <!-- frame -->
+        right below base_link origin; navigation stack depends on this frame -->
         <link name="base_footprint">
             <inertial>
@@ -17,22 +17,5 @@
                         izz="0.01"/>
             </inertial>
-            <visual>
-                <origin xyz="0 0 0" rpy="0 0 0"/>
-                <geometry>
-                    <box size="0.0 0.0 0.0"/>
-                </geometry>
-                <material name="Green"/>
-            </visual>
-            <collision>
-                <!-- represent base collision with a simple rectangular model,
-                <!-- positioned by base_size_z s.t. top surface of the collision
-                <!-- box matches the top surface of the PR2 base -->
-                <origin xyz="0 0 0" rpy="0 0 0"/>
-                <geometry>
-                    <box size="0.00 0.00 0.00"/>
-                </geometry>
-            </collision>
-        </link>
-        <!-- Base -->
+        </link>
         <!-- Links -->
         <link name="base_link">

File: segway_robot/urdf/sensors.urdf.xacro (robot description, xacro)
@@ -4,8 +4,8 @@
     <xacro:macro name="sensors" params="name">
         <!-- JOINT LIMIT VALUES FOR EFFORT AND VELOCITY NEED TO BE ADDED FOR
-        <!-- REVOLUTE AND CONTINUOUS JOINTS -->
+        REVOLUTE AND CONTINUOUS JOINTS -->
         <!-- Laser Base Laser -->
         <!-- Joint to world. Simply change the name and parent link when
-        <!-- attaching to own robot -->
+        attaching to own robot -->
         <joint name="base_laser_joint" type="fixed">
             <origin xyz="-0.057 0.010 0" rpy="1.57 0 3.14"/>
@@ -38,5 +38,5 @@
         <!-- Laser Tilt Laser -->
         <!-- Joint to world. Simply change the name and parent link when
-        <!-- attaching to own robot -->
+        attaching to own robot -->
         <joint name="tilt_laser_joint" type="fixed">
             <origin xyz="-0.056 -0.020 0" rpy="-1.57 0 3.14"/>
