Commit message: set proper parameters in segbot diff drive gazebo config et al

File: segway_robot/urdf/base.gazebo.xacro (robot description, xacro)
@@ -41,14 +41,18 @@
             <plugin name="differential_drive_controller" filename="libgazebo_ros_diff_drive.so">
                 <alwaysOn>true</alwaysOn>
-                <updateRate>1000.0</updateRate>
-                <leftJoint>segway_left_wheel_joint</leftJoint>
-                <rightJoint>segway_right_wheel_joint</rightJoint>
-                <wheelSeparation>0.544</wheelSeparation>
-                <wheelDiameter>1.35</wheelDiameter> <!-- TODO: measure -->
-                <torque>20</torque>
+                <updateRate>100.0</updateRate>
+                <rosDebugLevel>info</rosDebugLevel>
                 <commandTopic>cmd_vel</commandTopic>
                 <odometryTopic>odom</odometryTopic>
                 <odometryFrame>odom</odometryFrame>
                 <robotBaseFrame>base_footprint</robotBaseFrame>
+                <publishWheelTF>false</publishWheelTF>
+                <publishWheelJointState>false</publishWheelJointState>
+                <wheelSeparation>0.544</wheelSeparation>
+                <wheelDiameter>0.452574</wheelDiameter>
+                <odometrySource>world</odometrySource>
+                <leftJoint>segway_left_wheel_joint</leftJoint>
+                <rightJoint>segway_right_wheel_joint</rightJoint>
+                <publishTf>true</publishTf>
             </plugin>
             <plugin name="p3d_base_controller" filename="libgazebo_ros_p3d.so">

File: segway_robot/urdf/base.urdf.xacro (robot description, xacro)
@@ -305,5 +305,5 @@
         </joint>
         <joint name="segway_right_wheel_joint" type="continuous">
-            <origin xyz="-0.031 -0.353 -0.272" rpy="0 3.14 0"/>
+            <origin xyz="-0.031 -0.353 -0.272" rpy="0 0 0"/>
             <axis xyz="0 0 1"/>
             <limit effort="122" velocity="500"/>

File: segway_robot/urdf/sensors.gazebo.xacro (robot description, xacro)
@@ -6,5 +6,5 @@
                 <pose>0 0 0 0 0 0</pose>
                 <visualize>false</visualize>
-                <updateRate>20.0</updateRate>
+                <update_rate>20.0</update_rate>
                 <ray>
                     <scan>
@@ -29,5 +29,5 @@
                 <plugin name="gazebo_ros_base_laser_controller"
                         filename="libgazebo_ros_gpu_laser.so">
-                    <topicName>scan</topicName>
+                    <topicName>base_scan</topicName>
                     <frameName>base_laser_link</frameName>
                 </plugin>
@@ -38,5 +38,5 @@
                 <pose>0 0 0 0 0 0</pose>
                 <visualize>false</visualize>
-                <updateRate>20.0</updateRate>
+                <update_rate>20.0</update_rate>
                 <ray>
                     <scan>
@@ -61,6 +61,6 @@
                 <plugin name="gazebo_ros_tilt_laser_controller"
                         filename="libgazebo_ros_gpu_laser.so">
-                    <topicName>scan</topicName>
-                    <frameName>base_laser_link</frameName>
+                    <topicName>tilt_scan</topicName>
+                    <frameName>tilt_laser_link</frameName>
                 </plugin>
             </sensor>

Commit message: modify diff drive plugin to listen to ned transformed topic; lower mu for trailer wheel

File: segway_robot/urdf/base.gazebo.xacro (robot description, xacro)
@@ -19,4 +19,6 @@
         <gazebo reference="segway_trailer_wheel">
             <material>Gazebo/Red</material>
+            <mu1>0.2</mu1>
+            <mu2>0.2</mu2>
         </gazebo>
         <gazebo reference="battery_one">
@@ -43,5 +45,5 @@
                 <updateRate>100.0</updateRate>
                 <rosDebugLevel>info</rosDebugLevel>
-                <commandTopic>cmd_vel</commandTopic>
+                <commandTopic>cmd_vel_sim</commandTopic>
                 <odometryTopic>odom</odometryTopic>
                 <odometryFrame>odom</odometryFrame>

File: segway_robot/urdf/base.urdf.xacro (robot description, xacro)
@@ -147,5 +147,4 @@
                 <origin xyz="0 0 0" rpy="0 0 0"/>
                 <geometry name="segway_trailer_wheel_collision_geom">
-                    <!-- <mesh filename="package://segway_robot/meshes/convex/trailer_wheel_convex.stlb" /> -->
                     <cylinder radius="0.1285" length="0.097"/>
                 </geometry>
