Commit message: add  camera gazebo elements for front camera

File: segway_robot/urdf/sensors.gazebo.xacro (robot description, xacro)
@@ -68,4 +68,48 @@
             </sensor>
         </gazebo>
+        <gazebo reference="base_laser_link">
+            <sensor type="camera" name="${name}_sensor">
+                <update_rate>30.0</update_rate>
+                <camera name="segbot_cam">
+                    <horizontal_fov>1.5707</horizontal_fov>
+                    <image>
+                        <width>640</width>
+                        <height>480</height>
+                        <format>R8G8B8</format>
+                    </image>
+                    <clip>
+                        <near>0.01</near>
+                        <far>100.0</far>
+                    </clip>
+                    <noise>
+                        <type>gaussian</type>
+                        <!--
+                        Noise is sampled independently per pixel on each frame.
+                        That pixel's noise value is added to each of its color
+                        channels, which at that point lie in the range [0, 1].
+                        -->
+                        <mean>0.0</mean>
+                        <stddev>0.007</stddev>
+                    </noise>
+                </camera>
+                <plugin name="segbot_camera_gazebo_controller"
+                        filename="libgazebo_ros_camera.so">
+                    <robotNamespace>segbot</robotNamespace>
+                    <alwaysOn>true</alwaysOn>
+                    <updateRate>0.0</updateRate>
+                    <cameraName>segbot_cam</cameraName>
+                    <imageTopicName>image</imageTopicName>
+                    <cameraInfoTopicName>camera_info</cameraInfoTopicName>
+                    <frameName>base_laser_link</frameName>
+                    <hackBaseline>0.07</hackBaseline>
+                    <distortionK1>0.0</distortionK1>
+                    <distortionK2>0.0</distortionK2>
+                    <distortionK3>0.0</distortionK3>
+                    <distortionT1>0.0</distortionT1>
+                    <distortionT2>0.0</distortionT2>
+                </plugin>
+            </sensor>
+            <material>Gazebo/Green</material>
+        </gazebo>
     </xacro:macro>
 </robot>
