Commit message: add cylinder collision geometry to the top of the segbot for more accurate  detection with objects in gazebo

File: segway_robot/urdf/base.urdf.xacro (robot description, xacro)
@@ -40,4 +40,10 @@
                 </geometry>
             </collision>
+            <collision>
+                <origin xyz="-0.03164 0.12438 0.00167" rpy="1.5708 0 0"/>
+                <geometry name="segway_base_table_geom">
+                    <cylinder radius="0.3054" length="0.01587"/>
+                </geometry>
+            </collision>
         </link>
         <link name="segway_left_wheel">
