Commit message: add argument to segbot xacro to toggle gazebo namespacing

File: segbot_description/gazebo/gazebo.urdf.xacro (robot description, xacro)
@@ -4,5 +4,7 @@
         <static>false</static>
         <plugin name="gazebo_ros_control" filename="libgazebo_ros_control.so">
-            <robotNamespace>segbot</robotNamespace>
+            <xacro:if value="$(arg namespace)">
+                <robotNamespace>segbot</robotNamespace>
+            </xacro:if>
             <robotSimType>gazebo_ros_control/DefaultRobotHWSim</robotSimType>
         </plugin>

File: segbot_description/robots/segbot_without_arm.urdf.xacro (robot description, xacro)
@@ -1,9 +1,10 @@
 <?xml version="1.0"?>
 <robot name="segbot" xmlns:xacro="http://ros.org/wiki/xacro">
+    <xacro:arg name="namespace" default="false"/>
     <xacro:include filename="$(find segbot_description)/urdf/base.urdf.xacro"/>
     <xacro:include filename="$(find segbot_description)/urdf/sensors.urdf.xacro"/>
     <xacro:include filename="$(find segbot_description)/urdf/materials.xacro"/>
     <xacro:include filename="$(find segbot_description)/gazebo/gazebo.urdf.xacro"/>
-    <xacro:base name="base"/>
-    <xacro:sensors name="sensors"/>
+    <xacro:base name="base" namespace="$(arg namespace)"/>
+    <xacro:sensors name="sensors" namespace="$(arg namespace)"/>
 </robot>

File: segbot_description/urdf/base.gazebo.xacro (robot description, xacro)
@@ -1,5 +1,5 @@
 <?xml version="1.0"?>
 <robot xmlns:xacro="http://ros.org/wiki/xacro">
-    <xacro:macro name="base_gazebo" params="name">
+    <xacro:macro name="base_gazebo" params="name namespace">
         <gazebo reference="base_link">
             <material>Gazebo/Blue</material>
@@ -44,5 +44,7 @@
                 <alwaysOn>true</alwaysOn>
                 <updateRate>100.0</updateRate>
-                <robotNamespace>segbot</robotNamespace>
+                <xacro:if value="${namespace}">
+                    <robotNamespace>segbot</robotNamespace>
+                </xacro:if>
                 <rosDebugLevel>info</rosDebugLevel>
                 <commandTopic>cmd_vel_sim</commandTopic>
@@ -62,5 +64,7 @@
                 <alwaysOn>true</alwaysOn>
                 <updateRate>100.0</updateRate>
-                <robotNamespace>segbot</robotNamespace>
+                <xacro:if value="${namespace}">
+                    <robotNamespace>segbot</robotNamespace>
+                </xacro:if>
                 <bodyName>base_footprint</bodyName>
                 <topicName>base_pose_ground_truth</topicName>

File: segbot_description/urdf/base.transmission.xacro (robot description, xacro)
@@ -1,5 +1,5 @@
 <?xml version="1.0"?>
 <robot xmlns:xacro="http://ros.org/wiki/xacro">
-    <xacro:macro name="base_transmission" params="name">
+    <xacro:macro name="base_transmission" params="name namespace">
         <transmission name="segway_left_wheel_trans">
             <type>transmission_interface/SimpleTransmission</type>

File: segbot_description/urdf/base.urdf.xacro (robot description, xacro)
@@ -3,5 +3,5 @@
     <xacro:include filename="$(find segbot_description)/urdf/base.gazebo.xacro"/>
     <xacro:include filename="$(find segbot_description)/urdf/base.transmission.xacro"/>
-    <xacro:macro name="base" params="name">
+    <xacro:macro name="base" params="name namespace">
         <!-- JOINT LIMIT VALUES FOR EFFORT AND VELOCITY NEED TO BE ADDED FOR
         REVOLUTE AND CONTINUOUS JOINTS
@@ -378,6 +378,6 @@
             <calibration reference_position="0.0"/>
         </joint>
-        <xacro:base_gazebo name="${name}"/>
-        <xacro:base_transmission name="${name}"/>
+        <xacro:base_gazebo name="${name}" namespace="${namespace}"/>
+        <xacro:base_transmission name="${name}" namespace="${namespace}"/>
     </xacro:macro>
 </robot>

File: segbot_description/urdf/sensors.gazebo.xacro (robot description, xacro)
@@ -1,5 +1,5 @@
 <?xml version="1.0"?>
 <robot xmlns:xacro="http://ros.org/wiki/xacro">
-    <xacro:macro name="sensors_gazebo" params="name">
+    <xacro:macro name="sensors_gazebo" params="name namespace">
         <gazebo reference="base_laser_link">
             <sensor type="gpu_ray" name="base_laser">
@@ -29,5 +29,7 @@
                 <plugin name="gazebo_ros_base_laser_controller"
                         filename="libgazebo_ros_gpu_laser.so">
-                    <robotNamespace>segbot</robotNamespace>
+                    <xacro:if value="${namespace}">
+                        <robotNamespace>segbot</robotNamespace>
+                    </xacro:if>
                     <topicName>base_scan</topicName>
                     <frameName>base_laser_link</frameName>
@@ -62,5 +64,7 @@
                 <plugin name="gazebo_ros_tilt_laser_controller"
                         filename="libgazebo_ros_gpu_laser.so">
-                    <robotNamespace>segbot</robotNamespace>
+                    <xacro:if value="${namespace}">
+                        <robotNamespace>segbot</robotNamespace>
+                    </xacro:if>
                     <topicName>tilt_scan</topicName>
                     <frameName>tilt_laser_link</frameName>
@@ -95,5 +99,7 @@
                 <plugin name="segbot_camera_gazebo_controller"
                         filename="libgazebo_ros_camera.so">
-                    <robotNamespace>segbot</robotNamespace>
+                    <xacro:if value="${namespace}">
+                        <robotNamespace>segbot</robotNamespace>
+                    </xacro:if>
                     <alwaysOn>true</alwaysOn>
                     <updateRate>0.0</updateRate>

File: segbot_description/urdf/sensors.urdf.xacro (robot description, xacro)
@@ -2,5 +2,5 @@
 <robot xmlns:xacro="http://ros.org/wiki/xacro">
     <xacro:include filename="$(find segbot_description)/urdf/sensors.gazebo.xacro"/>
-    <xacro:macro name="sensors" params="name">
+    <xacro:macro name="sensors" params="name namespace">
         <!-- JOINT LIMIT VALUES FOR EFFORT AND VELOCITY NEED TO BE ADDED FOR
         REVOLUTE AND CONTINUOUS JOINTS -->
@@ -67,5 +67,5 @@
             </collision>
         </link>
-        <xacro:sensors_gazebo name="${name}"/>
+        <xacro:sensors_gazebo name="${name}" namespace="${namespace}"/>
     </xacro:macro>
 </robot>
