Commit message: remove dead segbot urdf element

File: segbot_description/urdf/base.urdf.xacro (robot description, xacro)
@@ -43,5 +43,4 @@
                 <origin xyz="-0.03164 0.132315 0.00167" rpy="1.5708 0 0"/>
                 <geometry name="segway_base_table_geom">
-<!--                    <cylinder radius="0.3054" length="0.01587"/> -->
                     <cylinder radius="0.4054" length="0.01587"/>
                 </geometry>

Commit message: replace trailer wheel collision model with sphere for better sim

File: segbot_description/urdf/base.urdf.xacro (robot description, xacro)
@@ -153,5 +153,5 @@
                 <origin xyz="0 0 0" rpy="0 0 0"/>
                 <geometry name="segway_trailer_wheel_collision_geom">
-                    <cylinder radius="0.1285" length="0.097"/>
+                    <sphere radius="0.1285"/>
                 </geometry>
             </collision>

Commit message: make a more robust landing platform collision model

File: segbot_description/urdf/base.urdf.xacro (robot description, xacro)
@@ -40,8 +40,35 @@
                 </geometry>
             </collision>
+            <!-- cover/expand the table on top of the segbot to (hopefully) -->
+            <!-- catch the hexacopter more robustly in simulation -->
             <collision>
                 <origin xyz="-0.03164 0.132315 0.00167" rpy="1.5708 0 0"/>
                 <geometry name="segway_base_table_geom">
-                    <cylinder radius="0.4054" length="0.01587"/>
+<!--                    <cylinder radius="0.4054" length="0.01587"/> -->
+                    <box size="0.8108 0.8108 0.01587"/>
+                </geometry>
+            </collision>
+            <collision>
+                <origin xyz="0.381535 0.17438 0.00167" rpy="0 0 0"/>
+                <geometry name="segway_base_basket_east">
+                    <box size="0.01587 0.1 0.8108"/>
+                </geometry>
+            </collision>
+            <collision>
+                <origin xyz="-0.444975 0.17438 0.00167" rpy="0 0 0"/>
+                <geometry name="segbot_base_basket_west">
+                    <box size="0.01587 0.1 0.8108"/>
+                </geometry>
+            </collision>
+            <collision>
+                <origin xyz="-0.03164 0.17438 0.415005" rpy="0 0 0"/>
+                <geometry name="segbot_base_basket_north">
+                    <box size="0.8108 0.1 0.01587"/>
+                </geometry>
+            </collision>
+            <collision>
+                <origin xyz="-0.03164 0.17438 -0.411665" rpy="0 0 0"/>
+                <geometry name="segbot_base_basket_south">>
+                    <box size="0.8108 0.1 0.01587"/>
                 </geometry>
             </collision>

Commit message: modify supposed calibration offset for mounted laser frame

File: segbot_description/urdf/base.urdf.xacro (robot description, xacro)
@@ -397,5 +397,5 @@
         </joint>
         <joint name="R313_hokuyo_laser2_joint" type="revolute">
-            <origin xyz="-0.162 0.283 0" rpy="1.57 -0.05 0" />
+            <origin xyz="-0.162 0.283 0" rpy="1.57 -0.01 0" />
             <axis xyz="0 0 1"/>
             <limit lower="-1.047" upper="1.047" effort="50" velocity="50"/>
