Commit message: remove null box geometry from segbot sensors

File: segbot_description/robots/segbot.urdf.xacro (robot description, xacro)
@@ -27,19 +27,4 @@
                iyy="0.01" iyz="0.0" izz="0.01" />
     </inertial>
-    <visual>
-      <origin xyz="0 0 0" rpy="0 0 0" />
-      <geometry>
-        <box size="0.0 0.0 0.0" />
-      </geometry>
-      <material name="Green" />
-    </visual>
-    <collision>
-      <!-- represent base collision with a simple rectangular model, positioned by base_size_z s.t. top
-           surface of the collision box matches the top surface of the PR2 base -->
-      <origin xyz="0 0 0" rpy="0 0 0" />
-      <geometry>
-        <box size="0.00 0.00 0.00" />
-      </geometry>
-    </collision>
   </link>
   <link name="base_link">
@@ -1248,17 +1233,4 @@
         <inertia ixx="0.0001" ixy="0" ixz="0" iyy="0.000001" iyz="0" izz="0.0001" />
       </inertial>
-      <visual>
-        <origin xyz="0 0 0" rpy="0 0 0" />
-        <geometry>
-          <box size="0.000 0.000 0.000" />
-        </geometry>
-        <material name="Red" />
-      </visual>
-      <collision>
-        <origin xyz="0 0 0" rpy="0 0 0" />
-        <geometry>
-          <box size=".000 .000 .00" />
-        </geometry>
-      </collision>
     </link>
 <!-- 			Actual laser		 -->
@@ -1300,17 +1272,4 @@
         <inertia ixx="0.0001" ixy="0" ixz="0" iyy="0.000001" iyz="0" izz="0.0001" />
       </inertial>
-      <visual>
-        <origin xyz="0 0 0" rpy="0 0 0" />
-        <geometry>
-          <box size="0 0 0" />
-        </geometry>
-        <material name="Red" />
-      </visual>
-      <collision>
-        <origin xyz="0 0 0" rpy="0 0 0" />
-        <geometry>
-          <box size="0 0 0" />
-        </geometry>
-      </collision>
     </link>
 <!-- 			Actual laser		 -->

File: segbot_description/urdf/sensors.urdf.xacro (robot description, xacro)
@@ -22,17 +22,4 @@
                          izz="0.0001"/>
             </inertial>
-            <visual>
-                <origin xyz="0 0 0" rpy="0 0 0"/>
-                <geometry>
-                    <box size="0.000 0.000 0.000"/>
-                </geometry>
-                <material name="Red"/>
-            </visual>
-            <collision>
-                <origin xyz="0 0 0" rpy="0 0 0"/>
-                <geometry>
-                    <box size="0.0 0.0 0.0"/>
-                </geometry>
-            </collision>
         </link>
         <!-- Laser Tilt Laser -->
@@ -53,17 +40,4 @@
                          izz="0.0001"/>
             </inertial>
-            <visual>
-                <origin xyz="0 0 0" rpy="0 0 0"/>
-                <geometry>
-                <box size="0 0 0"/>
-                </geometry>
-                <material name="Red"/>
-            </visual>
-            <collision>
-                <origin xyz="0 0 0" rpy="0 0 0"/>
-                <geometry>
-                    <box size="0 0 0"/>
-                </geometry>
-            </collision>
         </link>
         <xacro:sensors_gazebo name="${name}" namespace="${namespace}"/>
